File: Assets/PCB Files/.history/UGV.kicad_pcb (KiCad board)
At the start: 2 copper layers, 121 x 156.5 mm, 100 parts, among them J13 USB3_A, J15 Screw_Terminal_01x12, J16 Screw_Terminal_01x12, J17 Screw_Terminal_01x12, J18 Screw_Terminal_01x12, Q1 AO3400A, Q2 AO3400A, Q3 AO3400A, U2 LMR33630ADDA, U3 SN74LVC8T245, U4 Teensy4.1, U5 SN74LVC8T245

Commit message: Final PCB
Parts:
- removed D6: LED, LED_SMD:LED_1206_3216Metric_Pad1.42x1.75mm_HandSolder
- removed R12: 390 ohm, Resistor_SMD:R_1206_3216Metric_Pad1.30x1.75mm_HandSolder
- removed the REF** at (117.8, 5.73)
- removed the REF** at (22.5, 153.5)
- removed the REF** at (23.0, 5.55)
- removed the REF** at (118.0, 129.5)
- added Cout3: 22uF, Capacitor_SMD:C_1210_3225Metric_Pad1.33x2.70mm_HandSolder, F.Cu at (39.4, 129.4)
- added REF**: MountingHole_3.2mm_M3, MountingHole:MountingHole_3.2mm_M3, F.Cu at (117.7, 4.50)
- added REF**: MountingHole_3.2mm_M3, MountingHole:MountingHole_3.2mm_M3, F.Cu at (23.7, 154.0)
- added REF**: MountingHole_3.2mm_M3, MountingHole:MountingHole_3.2mm_M3, F.Cu at (117.7, 128.5)
- added REF**: MountingHole_3.2mm_M3, MountingHole:MountingHole_3.2mm_M3, F.Cu at (23.7, 4.50)
- R10: value 4.7 kohm -> 3.9 kohm
- U2: value LMR33630ADDA -> LMR33640ADDAR
- moved Q3 8.11 mm to (50.1, 67.2), turned to 90 degrees
- moved R6 4.94 mm to (47.0, 70.2), turned to -90 degrees
- moved D5 3.71 mm to (34.0, 133.5)
- moved R3 2.97 mm to (67.7, 127.7)
- moved Q1 2.97 mm to (72.2, 127.0)
- moved R2 2.97 mm to (70.4, 123.0)
- moved R7 2.89 mm to (51.1, 71.9), turned to 180 degrees
- moved Q2 2.40 mm to (76.7, 117.7)
- moved R5 2.40 mm to (76.0, 112.9)
- moved R4 2.40 mm to (80.0, 114.7)
- moved R11 2.05 mm to (30.0, 132.0), turned to 90 degrees
- moved Rfbt1 2.04 mm to (39.4, 124.3)
- moved Rfbb1 1.98 mm to (35.6, 121.6)
- moved Cff1 1.93 mm to (37.1, 124.9)
- moved Cout2 0.37 mm to (42.8, 129.4)
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- renumbered LED2 to StatusLED1
Routing:
- net /M1: track 16.0 -> 8.45 mm
- net GND: track 335.8 -> 342.4 mm
- net /Vin: track 59.8 -> 54.8 mm
- net /32: track 11.8 -> 15.9 mm
- net Net-(U2-FB): track 12.7 -> 15.9 mm
- net /Vout: track 223.3 -> 225.9 mm
- net /13: track 12.9 -> 15.5 mm
- net Net-(D6-K): track 2.24 -> 0.00 mm
- net Net-(Q2-D): track 54.5 -> 52.8 mm
- net /41: track 24.8 -> 23.2 mm
- net Net-(Q1-D): track 42.5 -> 41.2 mm
- net Net-(D5-K): track 2.24 -> 2.74 mm
