File: Assets/PCB Files/.history/UGV.kicad_sch (KiCad schematic)
At the start: 95 parts, among them J13 USB3_A, J15 Screw_Terminal_01x12, J16 Screw_Terminal_01x12, J17 Screw_Terminal_01x12, J18 Screw_Terminal_01x12, Q1 AO3400A, Q2 AO3400A, Q3 AO3400A, U2 LMR33630ADDA, U3 SN74LVC8T245, U4 Teensy4.1, U5 SN74LVC8T245

Commit message: Final PCB
Parts:
- removed D6: LED, LED_SMD:LED_1206_3216Metric_Pad1.42x1.75mm_HandSolder, symbol Device:LED
- removed R12: 390 ohm, Resistor_SMD:R_1206_3216Metric_Pad1.30x1.75mm_HandSolder, symbol Device:R
- added Cout3: 22uF, Capacitor_SMD:C_1210_3225Metric_Pad1.33x2.70mm_HandSolder, symbol Device:C
- R10: value 4.7 kohm -> 3.9 kohm
- U2: value LMR33630ADDA -> LMR33640ADDAR
- renumbered LED2 to StatusLED1
Connections:
- net GND: now also Cout3.2; no longer J13.SH (SHIELD)
- net Vout: now also Cout3.1
- no-connect marks 29 -> 30
Other:
- moved on the sheet: D5, R11
